File: smartdisplay.sch (KiCad schematic (older format))
At the start: 50 parts, among them J1 Conn_01x04_Female, J2 battery, J3 FPC24/0.5MM, Q1 Q_NMOS_DSG, U1 AMS1117-3.3, U2 ESP-32S, U3 DHT11, U4 FS8205, U5 tp4056, U6 DW01

Commit message: finish v1.0
Parts:
- removed C2, C4: 10uF, Diode_SMD:D_0603_1608Metric, symbol Device:C
- removed C6, C8: C, Capacitor_SMD:C_0603_1608Metric, symbol Device:C
- removed D1: LED, LED_SMD:LED_0603_1608Metric, symbol Device:LED
- removed FLASH1: FLASH, Button_Switch_SMD:SW_SPST_FSMSM, symbol Switch:SW_SPST
- removed H1, H2: MountingHole, MountingHole:MountingHole_2.2mm_M2, symbol Mechanical:MountingHole
- removed J1: Conn_01x04_Female, Connector_Wire:SolderWirePad_1x04_P3.81mm_Drill1mm, symbol Connector:Conn_01x04_Female
- removed J2: battery, Connector_JST:JST_PH_S2B-PH-K_1x02_P2.00mm_Horizontal, symbol Connector:Conn_01x02_Female
- removed J3: FPC24/0.5MM, smartdisplay:Hirose_FH12-24S-0.5SH_1x24-1MP_P0.50mm__redesign, symbol Connector_Generic:Conn_01x24
- removed R0: R, Resistor_SMD:R_0603_1608Metric, symbol Device:R
- removed U1: AMS1117-3.3, Package_TO_SOT_SMD:SOT-223-3_TabPin2, symbol Regulator_Linear:AMS1117-3.3
- removed U3: DHT11, Sensor:Aosong_DHT11_5.5x12.0_P2.54mm, symbol Sensor:DHT11
- removed U4: FS8205, Package_TO_SOT_SMD:SOT-23-6, symbol smartdisplay:FS8205
- removed U5: tp4056, Package_SO:SOP-8_3.9x4.9mm_P1.27mm, symbol smartdisplay:tp4056
- removed U6: DW01, Package_TO_SOT_SMD:TSOT-23-6, symbol smartdisplay:DW01
- removed USBC1: USB_C_Plug, Connector_USB:USB_C_Receptacle_Amphenol_12401548E4-2A, symbol Connector:USB_C_Plug
- added C17, C9: 1uF, Capacitor_SMD:C_0603_1608Metric, symbol Device:C
- added D3, D6: LED-red, Diode_SMD:D_0603_1608Metric, symbol Device:LED
- added J1, J3: Conn_01x01_Female, my:largepoint, symbol Connector:Conn_01x01_Female
- added J2: USB_C_Receptacle_USB2.0, Connector_USB:USB_C_Receptacle_HRO_TYPE-C-31-M-12, symbol Connector:USB_C_Receptacle_USB2.0
- added SW1: SW_Push, my:bt-342, symbol Switch:SW_Push
- added U1: DDC114TU-7-F, Package_TO_SOT_SMD:SOT-363_SC-70-6, symbol my:DDC114TU-7-F
- added U2: ch340k, my:ESSOP-10_3.9x4.9mm_P1.00mm, symbol my:ch340k
- added U3: 24pinconnecter, my:epd-24pin, symbol my:24pinconnecter
- added U5: SHT31-DIS, Sensor_Humidity:Sensirion_DFN-8-1EP_2.5x2.5mm_P0.5mm_EP1.1x1.7mm, symbol Sensor_Humidity:SHT31-DIS
- added U6: ME6211C33M5G-N, Package_TO_SOT_SMD:SOT-23-5, symbol my:ME6211C33M5G-N
- added U7: TP4054, Package_TO_SOT_SMD:SOT-23-5, symbol my:TP4054
- C1: renamed from C17; value 1uF/50V -> 1uF
- C10: renamed from C11; value 1uF/50V -> 1uF
- C11: renamed from C14; value 1uF/50V -> 1uF
- C12: renamed from C15; value 1uF/50V -> 1uF
- C13: renamed from C19; value 1uF/50V -> 1uF
- C14: renamed from C12; value 1uF/50V -> 1uF
- C15: renamed from C13; value 1uF/50V -> 1uF
- C16: value 1uF/50V -> 0.1uf
- C2: renamed from C18; value 1uF/50V -> 1uF
- C3: value 104 -> 0.1uf; footprint Diode_SMD:D_0603_1608Metric -> Capacitor_SMD:C_0603_1608Metric
- C4: renamed from C9; value 0.1uF/50V -> 4.7uF
- C5: value 104 -> 0.1uf
- C6: renamed from C1; value 10uF -> 1uF
- C7: renamed from C10; value 0.1uF/50V -> 1uF
- C8: renamed from C7; value 4.7uF/50V -> 4.7uF
- D1: renamed from D4; footprint Diode_SMD:D_0603_1608Metric -> Diode_SMD:D_SOD-123
- D2: value LED -> LED-green; footprint LED_SMD:LED_0603_1608Metric -> Diode_SMD:D_0603_1608Metric
- D4: renamed from D3; footprint Diode_SMD:D_0603_1608Metric -> Diode_SMD:D_SOD-123
- D5: footprint Diode_SMD:D_0603_1608Metric -> Diode_SMD:D_SOD-123
- L1: value 68uH -> 10uH; footprint Inductor_SMD:L_1812_4532Metric -> Inductor_SMD:L_Coilcraft_XxL4040
- Q1: value Q_NMOS_DSG -> SI1308EDL; symbol Device:Q_NMOS_DSG -> Device:Q_NMOS_GSD
- R1, R3: value 1k -> 10k
- R10, R6, R7, R8, R9: value R -> 10k
- R2: value 470 -> 10k
- R4: renamed from R11; value 10K -> 10k
- U4: renamed from U2; symbol ESP32-footprints-Shem-Lib:ESP-32S -> smartdisplay-rescue:ESP-32S-ESP32-footprints-Shem-Lib
- renumbered R12 to R5
Connections:
- net labels added: +3.3V, +5V, BAT+, D+, D-, DTR, RTS, SCL, SCLK, SDA
- net labels removed: B+, B-, BAT, BS, CLK, IO16, IO2, OC, OD, OUT+, OUT-, S2, USB5V, VDD3.3V, VDD3V3
- wire segments 166 -> 113
- no-connect marks 37 -> 32
Other:
- note added: "EPAPER"
- note added: "ESP32"
- note added: "POWER"
- note added: "TEMP"
- note added: "USB-TTL"
- note removed: "1.EPAPER"
- note removed: "2.KEY\n"
- note removed: "3.MCU"
- note removed: "4.POWER"
- note removed: "5.SENSOR"
- note removed: "6.hole"
- note removed: "connector"
- moved on the sheet: C1, C10, C11, C12, C13, C14, C15, C2, C4, C6, C7, C8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
